Commit message: Renamed frames with azure_kinect prefix

File: azure_kinect_ros_driver/urdf/azure_kinect.urdf.xacro (robot description, xacro)
@@ -17,5 +17,7 @@
     <color rgba="0.9 0.9 0.9 1" />
   </material>
-  <link name="camera_body">
+  <!-- Define tf_prefix -->
+  <xacro:property name="tf_prefix" value="azure_kinect" />
+  <link name="${tf_prefix}_camera_body">
     <visual>
       <origin xyz="0. 0. 0." />
@@ -26,5 +28,5 @@
     </visual>
   </link>
-  <link name="camera_base">
+  <link name="${tf_prefix}_camera_base">
     <visual>
       <origin xyz="-0.013 0. 0." />
@@ -35,5 +37,5 @@
     </visual>
   </link>
-  <link name="camera_visor">
+  <link name="${tf_prefix}_camera_visor">
     <visual>
       <origin xyz="-0.0128 0. 0." />
@@ -45,11 +47,11 @@
   </link>
   <joint name="camera_base_to_body" type="fixed">
-    <parent link="camera_base" />
-    <child link="camera_body" />
+    <parent link="${tf_prefix}_camera_base" />
+    <child link="${tf_prefix}_camera_body" />
     <origin xyz="-0.0757 0. 0.008" rpy="0. 0. 0." />
   </joint>
   <joint name="camera_base_to_visor" type="fixed">
-    <parent link="camera_base" />
-    <child link="camera_visor" />
+    <parent link="${tf_prefix}_camera_base" />
+    <child link="${tf_prefix}_camera_visor" />
     <origin xyz="0. 0. 0." rpy="0. 0. 0." />
   </joint>

Commit message: Legacy support

File: azure_kinect_ros_driver/urdf/azure_kinect.urdf.xacro (robot description, xacro)
@@ -18,6 +18,5 @@
   </material>
   <!-- Define tf_prefix -->
-  <xacro:property name="tf_prefix" value="azure_kinect" />
-  <link name="${tf_prefix}_camera_body">
+  <link name="camera_body">
     <visual>
       <origin xyz="0. 0. 0." />
@@ -28,5 +27,5 @@
     </visual>
   </link>
-  <link name="${tf_prefix}_camera_base">
+  <link name="camera_base">
     <visual>
       <origin xyz="-0.013 0. 0." />
@@ -47,11 +46,11 @@
   </link>
   <joint name="camera_base_to_body" type="fixed">
-    <parent link="${tf_prefix}_camera_base" />
-    <child link="${tf_prefix}_camera_body" />
+    <parent link="camera_base" />
+    <child link="camera_body" />
     <origin xyz="-0.0757 0. 0.008" rpy="0. 0. 0." />
   </joint>
   <joint name="camera_base_to_visor" type="fixed">
-    <parent link="${tf_prefix}_camera_base" />
-    <child link="${tf_prefix}_camera_visor" />
+    <parent link="camera_base" />
+    <child link="camera_visor" />
     <origin xyz="0. 0. 0." rpy="0. 0. 0." />
   </joint>
